Commit message: Added revised launch files and cad models

File: trilobyte_description/urdf/trilobyte.urdf (robot description, URDF)
Before this commit: robot trilobyte, 1 links, 0 joints
Links:
- link base_link: geometry visual mesh filename=package://trilobyte_description/meshes/trilobyte_base_link.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 scale=0.001 0.001 0.001
