Commit message: Added hardware folder to docker

File: trilobyte_description/urdf/trilobyte.urdf.xacro (robot description, xacro)
@@ -1,4 +1,20 @@
 <?xml version="1.0"?>
 <robot xmlns:xacro="http://www.ros.org/wiki/xacro"  name="trilobyte">
+      <!-- Constants for robot dimensions -->
+    <xacro:property name="PI" value="3.1415926535897931"/>
+    <xacro:property name="base_mass" value="0.3" /> <!-- arbitrary value for base mass -->
+    <xacro:property name="base_width" value="0.1" />
+    <xacro:property name="base_length" value="0.1" />
+    <xacro:property name="base_height" value="0.05" />
+    <xacro:property name="wheel_mass" value="0.3" /> <!-- arbitrary value for wheel mass -->
+    <xacro:property name="wheel_len" value="0.020" />
+    <xacro:property name="wheel_radius" value="0.015" />
+    <xacro:property name="caster_wheel_mass" value="0.1" /> <!-- arbitrary value for caster wheel mass -->
+    <xacro:property name="caster_wheel_radius" value="0.015" />
+    <xacro:property name="z_offset" value="-${base_height/2}" /> <!-- Space btw top of beam and the each joint -->
+    <!-- Core Robot Description -->
     <xacro:include filename="trilobyte_core.xacro" />
+    <!-- ROS2 Control -->
+    <xacro:include filename="$(find trilobyte_hardware_interface)/ros2_control/trilobyte_ros2_control.xacro" />
+    <xacro:trilobyte_ros2_control name="trilobyte" />
 </robot>

Commit message: changes to trilbyte hardware and description

File: trilobyte_description/urdf/trilobyte.urdf.xacro (robot description, xacro)
@@ -12,9 +12,8 @@
     <xacro:property name="caster_wheel_mass" value="0.1" /> <!-- arbitrary value for caster wheel mass -->
     <xacro:property name="caster_wheel_radius" value="0.015" />
-    <xacro:property name="z_offset" value="-${base_height/2}" /> <!-- Space btw top of beam and the each joint -->
     <!-- Core Robot Description -->
     <xacro:include filename="trilobyte_core.xacro" />
     <!-- ROS2 Control -->
-    <xacro:include filename="$(find trilobyte_hardware_interface)/ros2_control/trilobyte_ros2_control.xacro" />
+    <xacro:include filename="$(find trilobyte_hardware_interface)/description/trilobyte_ros2_control.xacro" />
     <xacro:trilobyte_ros2_control name="trilobyte" />
 </robot>

File: trilobyte_hardware_interface/description/trilobyte_ros2_control.xacro (robot description, xacro)
@@ -10,12 +10,19 @@
         <joint name="joint_wheel_left">
           <command_interface name="velocity">
-            <!-- <param name="min">{-2*pi}</param>
-            <param name="max">{2*pi}</param> -->
           </command_interface>
-          <!-- additional command interfaces ... -->
+          <state_interface name="position">
+          </state_interface>
           <state_interface name="velocity">
             <param name="initial_value">0.0</param>
           </state_interface>
-          <!-- additional state interfaces ... -->
+        </joint>
+        <joint name="joint_wheel_right">
+          <command_interface name="velocity">
+          </command_interface>
+          <state_interface name="position">
+          </state_interface>
+          <state_interface name="velocity">
+            <param name="initial_value">0.0</param>
+          </state_interface>
         </joint>
         <!-- additional joints ...-->
