Commit message: corrected urdf for base footprint transform

File: trilobyte_description/urdf/trilobyte_core.xacro (robot description, xacro)
@@ -3,6 +3,6 @@
   <link name="base_footprint" />
   <joint name="base_joint" type="fixed">
-    <parent link="base_footprint" />
-    <child link="base_link" />
+    <parent link="base_link" />
+    <child link="base_footprint" />
     <origin xyz="0 0 0.05" rpy="0 0 0" />
   </joint>

Commit message: not quite working vel and pos

File: trilobyte_description/urdf/trilobyte_core.xacro (robot description, xacro)
@@ -43,5 +43,5 @@
     <child link="wheel_right" />
     <origin xyz="0 -0.12 0" rpy="0 0 0" />
-    <axis xyz= "0 -1 0" />
+    <axis xyz= "0 1 0" />
   </joint>
   <!-- Caster Wheel -->

Commit message: added slam toolbox, prelininary tests of mapping

File: trilobyte_description/urdf/trilobyte_core.xacro (robot description, xacro)
@@ -60,3 +60,10 @@
     <!-- <axis xyz= "0 0 0" /> -->
   </joint>
+  <link name="base_laser">
+  </link>
+ <joint name="joint_base_laser" type="fixed">
+  <parent link="base_link" />
+  <child link="base_laser" />
+  <origin xyz="0 0.06 0.12" rpy="0 0 0" />
+ </joint>
 </robot>

Commit message: Added hardware changes for gripper

File: trilobyte_description/urdf/trilobyte_core.xacro (robot description, xacro)
@@ -14,4 +14,31 @@
             </geometry>
     </visual>
+  </link>
+  <joint name="joint_base_lifter" type="revolute">
+    <parent link="base_link" />
+    <child link="lifter" />
+    <limit effort="10.0" velocity="5.0" />
+  </joint>
+  <joint name="joint_lifter_gripper_left" type="revolute">
+    <parent link="lifter" />
+    <child link="gripper_left" />
+    <limit effort="10.0" velocity="5.0" />
+  </joint>
+  <joint name="joint_lifter_gripper_right" type="revolute">
+    <parent link="lifter" />
+    <child link="gripper_right" />
+    <limit effort="10.0" velocity="5.0" />
+  </joint>
+  <link name="lifter">
+    <visual>
+      <origin xyz="0.0 0.0 0.02" rpy="0 0 1.57" />
+      <geometry>
+          <mesh filename="package://trilobyte_description/meshes/lifter.obj"/>
+      </geometry>
+    </visual>
+  </link>
+  <link name="gripper_left">
+  </link>
+  <link name = "gripper_right">
   </link>
   <!-- Left Wheel -->

File: trilobyte_hardware_interface/description/trilobyte_ros2_control.xacro (robot description, xacro)
@@ -8,5 +8,6 @@
             <param name="right_wheel_name">joint_wheel_right</param>
             <param name="loop_rate">30</param>
-            <param name="device">/dev/ttyACM0</param>
+            <param name="device_pico">/dev/ttyACM0</param>
+            <param name="device_esp">/dev/ttyUSB1</param>
             <param name="baud_rate">115200</param>
             <param name="timeout">1000</param>

Commit message: Edits to urdf.

File: trilobyte_description/urdf/trilobyte_core.xacro (robot description, xacro)
@@ -18,4 +18,5 @@
     <parent link="base_link" />
     <child link="lifter" />
+    <origin xyz="0 0 0" rpy="0 0 0" />
     <limit effort="10.0" velocity="5.0" />
   </joint>
@@ -23,4 +24,5 @@
     <parent link="lifter" />
     <child link="gripper_left" />
+    <origin xyz="0 0 0" rpy="0 0 0" />
     <limit effort="10.0" velocity="5.0" />
   </joint>
@@ -28,4 +30,5 @@
     <parent link="lifter" />
     <child link="gripper_right" />
+    <origin xyz="0 0 0" rpy="0 0 0" />
     <limit effort="10.0" velocity="5.0" />
   </joint>

Commit message: Added some ros2 control config for gripper

File: trilobyte_description/urdf/trilobyte_core.xacro (robot description, xacro)
@@ -21,10 +21,10 @@
     <limit effort="10.0" velocity="5.0" />
   </joint>
-  <joint name="joint_lifter_gripper_left" type="revolute">
+  <!-- <joint name="joint_lifter_gripper_left" type="revolute">
     <parent link="lifter" />
     <child link="gripper_left" />
     <origin xyz="0 0 0" rpy="0 0 0" />
     <limit effort="10.0" velocity="5.0" />
-  </joint>
+  </joint> -->
   <joint name="joint_lifter_gripper_right" type="revolute">
     <parent link="lifter" />

File: trilobyte_hardware_interface/description/trilobyte_ros2_control.xacro (robot description, xacro)
@@ -33,4 +33,20 @@
           <state_interface name="position"/>
         </joint>
+        <joint name="joint_base_lifter">
+          <command_interface name="position">
+            <param name="min">0</param>
+            <param name="max">4095</param>
+          </command_interface>
+          <state_interface name="position"/>
+          <state_interface name="load"/>
+        </joint>
+        <joint name="joint_lifter_gripper_right">
+          <command_interface name="position">
+            <param name="min">0</param>
+            <param name="max">4095</param>
+          </command_interface>
+          <state_interface name="position"/>
+          <state_interface name="load"/>
+        </joint>
         <!-- additional joints ...-->
         <!-- additional hardware/sensors ...-->

Commit message: Added radians command to position on servos, and set limits.

File: trilobyte_description/urdf/trilobyte_core.xacro (robot description, xacro)
@@ -19,5 +19,16 @@
     <child link="lifter" />
     <origin xyz="0 0 0" rpy="0 0 0" />
-    <limit effort="10.0" velocity="5.0" />
+    <axis xyz="0 0 1"/>
+    <limit lower="-1.0" upper="1.0" effort="1.0" velocity="1.0" />
+    <transmission name="joint_base_lifter_trans">
+    <type>transmission_interface/SimpleTransmission</type>
+    <actuator name="lifter_motor">
+      <mechanicalReduction>1</mechanicalReduction>
+    </actuator>
+  </transmission>
+    <sensor name="sensor_lifter_load">
+      <origin xyz="0 0 0" rpy="0 0 0" />
+      <parent>lifter</parent>
+    </sensor>
   </joint>
   <!-- <joint name="joint_lifter_gripper_left" type="revolute">
@@ -31,5 +42,16 @@
     <child link="gripper_right" />
     <origin xyz="0 0 0" rpy="0 0 0" />
-    <limit effort="10.0" velocity="5.0" />
+    <axis xyz="0 0 1"/>
+    <limit lower="-1.0" upper="1.0" effort="1.0" velocity="1.0" />
+    <transmission name="joint_lifter_gripper_right_trans">
+    <type>transmission_interface/SimpleTransmission</type>
+    <actuator name="gripper_motor">
+      <mechanicalReduction>1</mechanicalReduction>
+    </actuator>
+  </transmission>
+    <sensor name="sensor_gripper_load">
+      <origin xyz="0 0 0" rpy="0 0 0" />
+      <parent>gripper_right</parent>
+    </sensor>
   </joint>
   <link name="lifter">
@@ -41,6 +63,6 @@
     </visual>
   </link>
-  <link name="gripper_left">
-  </link>
+  <!-- <link name="gripper_left">
+  </link> -->
   <link name = "gripper_right">
   </link>

File: trilobyte_hardware_interface/description/trilobyte_ros2_control.xacro (robot description, xacro)
@@ -39,5 +39,4 @@
           </command_interface>
           <state_interface name="position"/>
-          <state_interface name="load"/>
         </joint>
         <joint name="joint_lifter_gripper_right">
@@ -47,5 +46,4 @@
           </command_interface>
           <state_interface name="position"/>
-          <state_interface name="load"/>
         </joint>
         <!-- additional joints ...-->

Commit message: adding camera

File: trilobyte_description/urdf/trilobyte_core.xacro (robot description, xacro)
@@ -113,4 +113,5 @@
   </joint>
   <link name="base_laser">
+    <origin xyz="0.0 0.06 0.12" rpy="0 0 3.14"/>
   </link>
  <joint name="joint_base_laser" type="fixed">
