Commit message: fixed hardware interface connections, working

File: trilobyte_hardware_interface/description/trilobyte_ros2_control.xacro (robot description, xacro)
@@ -1,10 +1,11 @@
- <?xml version="1.0"?>
-<robot xmlns:xacro="http://www.ros.org/wiki/xacro">
-  <xacro:macro name="trilobyte_ros2_control" params="name prefix">
+<?xml version="1.0"?>
+<robot xmlns:xacro="http://www.ros.org/wiki/xacro" name="trilobyte">
+  <xacro:macro name="trilobyte_ros2_control" params="name">
     <ros2_control name="${name}" type="system">
         <hardware>
-          <plugin>
-            <!-- {Name_Space}/{Class_Name}-->
-          </plugin>
+          <plugin>trilobyte_hardware_interface/TrilobyteControlSystem</plugin>
+          <param name="example_param_hw_start_duration_sec">0.0</param>
+          <param name="example_param_hw_stop_duration_sec">3.0</param>
+          <param name="example_param_hw_slowdown">10.0</param>
         </hardware>
         <joint name="joint_wheel_left">
